File: k3ng_cw_keyer.sch (KiCad schematic (older format))
At the start: 51 parts, among them J1 Jack-DC, J2 Conn_01x06, J3 Conn_01x03, J4 Conn_01x04, J5 Mini-DIN-6, J6 AJ-1780, J7 AJ-1780, J8 AJ-1780, Q1 Q_NPN_BCE, SW1 SW_Push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

Commit message: Update MiniDin-6
Parts:
- removed J5: Mini-DIN-6, Connectors_JST:JST_ZE_S06B-ZESK-2D_06x1.5mm_Angled, symbol Mini-DIN-6
- added J5: MJ373-6, module:MJ373-6, symbol MJ373-6
- J6, J7, J8: footprint (none) -> module:AJ-1780
Connections:
- net +5V: now also J5.4
- net GND: now also J5.3
- net at L1.1: now also J5.1
- net at L2.1: now also J5.5
Changed lines of the file:
@@
-$EndComp
-$Comp
-L Mini-DIN-6 J5
-U 1 1 59DEFB9A
-P 9400 5050
-F 0 "J5" H 9400 5300 50  0000 C CNN
-F 1 "Mini-DIN-6" H 9400 4800 50  0000 C CNN
-F 2 "Connectors_JST:JST_ZE_S06B-ZESK-2D_06x1.5mm_Angled" H 9400 5050 50  0001 C CNN
-F 3 "" H 9400 5050 50  0001 C CNN
-	1    9400 5050
-	-1   0    0    1
 $EndComp
 $Comp
@@
 	5400 6300 5400 6500
 Wire Wire Line
-	5200 2150 5200 2300
+	5200 2150 5200 2200
+Wire Wire Line
+	5200 2200 5200 2300
 Connection ~ 4250 3000
 Connection ~ 4250 3400
@@
 	3750 3000 3700 3000
 Wire Wire Line
-	3700 3000 3700 3400
+	3700 3000 3700 3200
+Wire Wire Line
+	3700 3200 3700 3400
 Wire Wire Line
 	3700 3400 3750 3400
@@
 	6050 2200 5850 2200
 Wire Wire Line
-	5200 2200 5550 2200
+	5200 2200 5400 2200
+Wire Wire Line
+	5400 2200 5550 2200
 Connection ~ 5400 2200
 Connection ~ 5200 2200
@@
 	3900 2150 3900 2050
 Wire Wire Line
-	3900 1600 3900 1750
+	3900 1600 3900 1700
+Wire Wire Line
+	3900 1700 3900 1750
 Connection ~ 3900 2150
 Wire Wire Line
-	3500 2150 4200 2150
-Wire Wire Line
-	7600 5800 7950 5800
+	3500 2150 3600 2150
+Wire Wire Line
+	3600 2150 3900 2150
+Wire Wire Line
+	3900 2150 4200 2150
+Wire Wire Line
+	7600 5800 7800 5800
+Wire Wire Line
+	7800 5800 7950 5800
 Wire Wire Line
 	7700 5600 7950 5600
@@
 	6400 5600 7400 5600
 Wire Wire Line
-	8750 5600 9600 5600
-Wire Wire Line
-	8750 5800 9600 5800
-Wire Wire Line
-	8750 6250 9600 6250
-Wire Wire Line
-	8750 6450 9600 6450
-Wire Wire Line
-	9200 1150 9200 1250
-Wire Wire Line
-	9200 1550 9200 1650
-Wire Wire Line
-	9200 1950 9200 2050
-Wire Wire Line
-	9200 2350 9200 2450
+	8750 5600 9000 5600
+Wire Wire Line
+	9000 5600 9600 5600
+Wire Wire Line
+	8750 5800 9000 5800
+Wire Wire Line
+	9000 5800 9600 5800
+Wire Wire Line
+	8750 6250 9000 6250
+Wire Wire Line
+	9000 6250 9600 6250
+Wire Wire Line
+	8750 6450 9000 6450
+Wire Wire Line
+	9000 6450 9600 6450
+Wire Wire Line
+	9200 1150 9200 1200
+Wire Wire Line
+	9200 1200 9200 1250
+Wire Wire Line
+	9200 1550 9200 1600
+Wire Wire Line
+	9200 1600 9200 1650
+Wire Wire Line
+	9200 1950 9200 2000
+Wire Wire Line
+	9200 2000 9200 2050
+Wire Wire Line
+	9200 2350 9200 2400
+Wire Wire Line
+	9200 2400 9200 2450
 Wire Wire Line
 	9200 2750 9200 2800
@@
 Connection ~ 9200 1600
 Wire Wire Line
-	9950 1200 9950 2950
+	9950 1200 9950 1600
+Wire Wire Line
+	9950 1600 9950 2000
+Wire Wire Line
+	9950 2000 9950 2400
+Wire Wire Line
+	9950 2400 9950 2800
+Wire Wire Line
+	9950 2800 9950 2950
 Wire Wire Line
 	9950 1200 9800 1200
@@
 	8750 4500 8750 4550
 Wire Wire Line
-	6400 3700 9600 3700
-Wire Wire Line
-	7150 3800 9600 3800
+	6400 3700 8050 3700
+Wire Wire Line
+	8050 3700 9600 3700
+Wire Wire Line
+	7150 3800 8300 3800
+Wire Wire Line
+	8300 3800 9600 3800
 Wire Wire Line
 	4150 4150 4150 4200
@@
 	1850 2650 1850 2750
 Wire Wire Line
-	1600 2150 3200 2150
+	1600 2150 3050 2150
+Wire Wire Line
+	3050 2150 3200 2150
 Text Notes 9150 4250 0    60   ~ 0
 SCL\n
@@
 	6950 3900 6400 3900
 Wire Wire Line
-	7700 2600 7700 2700
+	7700 2600 7700 2650
+Wire Wire Line
+	7700 2650 7700 2700
 Wire Wire Line
 	7700 2250 7700 2300
@@
 USB5V
 Wire Wire Line
-	1900 5300 2350 5300
+	1900 5300 1950 5300
+Wire Wire Line
+	1950 5300 2200 5300
+Wire Wire Line
+	2200 5300 2350 5300
 Wire Wire Line
 	1950 5350 1950 5300
@@
 Connection ~ 2200 5300
 Wire Wire Line
-	2950 5300 3750 5300
+	2950 5300 3100 5300
+Wire Wire Line
+	3100 5300 3750 5300
 Wire Wire Line
 	3750 5500 3550 5500
@@
 	1550 5300 1600 5300
 Wire Wire Line
-	1550 5400 1550 5650
+	1550 5400 1550 5500
+Wire Wire Line
+	1550 5500 1550 5650
 Connection ~ 1550 5500
 NoConn ~ 6400 2800
@@
 	7150 2700 7150 1200
 Wire Wire Line
-	7150 1200 9400 1200
+	7150 1200 9200 1200
+Wire Wire Line
+	9200 1200 9400 1200
 $Comp
 L POT RV1
@@
 $EndComp
 Wire Wire Line
-	4200 2050 4200 2600
+	4200 2050 4200 2150
+Wire Wire Line
+	4200 2150 4200 2600
 Connection ~ 4200 2150
 Wire Wire Line
@@
 	3050 2500 3050 2650
 Wire Wire Line
-	4050 3000 4400 3000
-Wire Wire Line
-	4050 3400 4400 3400
+	4050 3000 4250 3000
+Wire Wire Line
+	4250 3000 4400 3000
+Wire Wire Line
+	4050 3400 4250 3400
+Wire Wire Line
+	4250 3400 4400 3400
 $Comp
 L R R1
@@
 F 0 "J7" H 9800 5890 50  0000 C CNN
 F 1 "AJ-1780" H 9650 5350 50  0000 L CNN
-F 2 "" H 10050 5700 50  0001 C CNN
+F 2 "module:AJ-1780" H 10050 5700 50  0001 C CNN
 F 3 "" H 10050 5700 50  0001 C CNN
 	1    9800 5600
@@
 F 0 "J8" H 9800 6540 50  0000 C CNN
 F 1 "AJ-1780" H 9650 6000 50  0000 L CNN
-F 2 "" H 10050 6350 50  0001 C CNN
+F 2 "module:AJ-1780" H 10050 6350 50  0001 C CNN
 F 3 "" H 10050 6350 50  0001 C CNN
 	1    9800 6250
@@
 F 0 "J6" H 9800 4090 50  0000 C CNN
 F 1 "AJ-1780" H 9650 3550 50  0000 L CNN
-F 2 "" H 10050 3900 50  0001 C CNN
+F 2 "module:AJ-1780" H 10050 3900 50  0001 C CNN
 F 3 "" H 10050 3900 50  0001 C CNN
 	1    9800 3800
@@
 NoConn ~ 9600 3600
 NoConn ~ 9600 3900
+$Comp
+L MJ373-6 J5
+U 1 1 5ACEE3C3
+P 9400 5050
+F 0 "J5" H 9400 5300 50  0000 C CNN
+F 1 "MJ373-6" H 9400 4800 50  0000 C CNN
+F 2 "module:MJ373-6" H 9400 5050 50  0001 C CNN
+F 3 "" H 9400 5050 50  0001 C CNN
+	1    9400 5050
+	-1   0    0    1
+$EndComp
 $EndSCHEMATC

Commit message: KiCAD 5
Parts:
- C1, C3, C9: symbol CP_Small -> Device:CP_Small
- C10, C11, C12, C13, C2: symbol C_Small -> Device:C_Small
- C4, C5, C6, C7, C8: symbol C -> Device:C
- D1, D2: symbol D -> Device:D
- J1: symbol Jack-DC -> k3ng_cw_keyer-rescue:Jack-DC
- J2: symbol Conn_01x06 -> k3ng_cw_keyer-rescue:Conn_01x06
- J3: symbol Conn_01x03 -> k3ng_cw_keyer-rescue:Conn_01x03
- J4: symbol Conn_01x04 -> k3ng_cw_keyer-rescue:Conn_01x04
- J5: symbol MJ373-6 -> MJ373:MJ373-6
- J6, J7, J8: symbol AJ-1780 -> AJ-1780:AJ-1780
- L1, L2: symbol Ferrite_Bead -> Device:Ferrite_Bead
- LS1: symbol Speaker -> Device:Speaker
- Q1: symbol Q_NPN_BCE -> Device:Q_NPN_BCE
- R1, R10, R11, R12, R13, R2, R3, R4, R5, R6, R7, R8, R9: symbol R -> Device:R
- RV1: symbol POT -> k3ng_cw_keyer-rescue:POT
- SW1, SW2, SW3, SW4, SW5, SW6: symbol SW_Push -> k3ng_cw_keyer-rescue:SW_Push
- U1: symbol L7805 -> k3ng_cw_keyer-rescue:L7805
- U2: symbol ATMEGA1284-PU -> k3ng_cw_keyer-rescue:ATMEGA1284-PU
- U3: symbol TLP627-2 -> k3ng_cw_keyer-rescue:TLP627-2
- Y1: symbol Crystal -> Device:Crystal
